Commit message: Pincher MK3 Updates. New IKFast solver.

File: phantomx_pincher_arm_description/urdf/arm_hardware.xacro (robot description, xacro)
@@ -3,53 +3,12 @@
 <robot xmlns:xacro="http://ros.org/wiki/xacro">
   <xacro:property name="M_PI" value="3.14159"/>
-  <xacro:property name="M_SCALE" value="0.001"/>
-  <xacro:property name="F10_HEIGHT" value="0.004"/>
-  <xacro:property name="F4_HEIGHT" value="0.0525"/>
-  <xacro:property name="F3_HEIGHT" value="0.009"/>
-  <xacro:property name="AX12_HEIGHT" value="0.0385"/>
-  <xacro:property name="AX12_WIDTH" value="0.038"/>
-  <xacro:property name="AX12_LENGTH" value="0.050"/>
-  <xacro:property name="F2_HEIGHT" value="0.0265"/>
-  <xacro:macro name="arm_mount" params="parent name color *origin">
+  <xacro:macro name="pincher_base" params="parent name *origin">
     <joint name="${name}_joint" type="fixed">
-      <insert_block name="origin"/>
-      <parent link="${parent}"/>
-      <child link="${name}_link"/>
-    </joint>
-    <link name="${name}_link">
-      <inertial>
-        <mass value="0.018"/>
-        <origin xyz="0 0 0"/>
-        <inertia ixx="0.000001" ixy="0.0" ixz="0.0"
-                 iyy="0.000001" iyz="0.0"
-                 izz="0.000001"/>
-      </inertial>
-      <visual>
-        <origin xyz="-0.028 -0.0493 0.014" rpy="0.0 0.0 -${M_PI/2}"/>
-        <geometry>
-          <mesh filename="package://phantomx_pincher_arm_description/meshes/mount.stl" scale="${M_SCALE} ${M_SCALE} ${M_SCALE}"/>
-        </geometry>
-        <material name="${color}"/>
-      </visual>
-      <collision>
-        <origin xyz="-0.01 0.0 0.0165" rpy="0.0 0.0 0.0"/>
-        <geometry>
-          <box size="0.074 0.074 0.004"/>
-        </geometry>
-      </collision>
-    </link>
-    <gazebo reference="${name}_link">
-      <material>Gazebo/${color}</material>
-      <selfCollide>true</selfCollide>
-      <gravity>true</gravity>
-    </gazebo>
-  </xacro:macro>
-  <xacro:macro name="dynamixel_AX12_fixed" params="parent name *origin">
-    <joint name="${name}_joint" type="fixed">
-      <insert_block name="origin"/>
-      <parent link="${parent}"/>
-      <child link="${name}_link"/>
-    </joint>
-    <link name="${name}_link">
+      <xacro:insert_block name="origin"/>
+      <parent link="${parent}"/>
+      <child link="${name}_link"/>
+    </joint>
+    <link name="${name}_link">
+      <!-- TODO: This inertial field needs doesn't contain reliable data!! -->
       <inertial>
         <mass value="0.055"/>
@@ -60,32 +19,109 @@
       </inertial>
       <visual>
+        <origin xyz="0 0 0" rpy="0 0 0"/>
+        <geometry>
+          <mesh filename="package://phantomx_pincher_arm_description/meshes/PincherBase.stl" scale="1.0 1.0 1.0"/>
+        </geometry>
+        <material name="Black"/>
+      </visual>
+      <collision>
+        <origin xyz="0 0 0" rpy="0 0 0"/>
+        <geometry>
+          <mesh filename="package://phantomx_pincher_arm_description/meshes/PincherBase.stl" scale="1.0 1.0 1.0"/>
+        </geometry>
+      </collision>
+    </link>
+    <gazebo reference="${name}_link">
+      <material>Gazebo/Black</material>
+      <gravity>true</gravity>
+    </gazebo>
+  </xacro:macro>
+  <xacro:macro name="bracket_F2_revolute" params="parent name color llimit ulimit vlimit *origin">
+    <joint name="${name}_joint" type="revolute">
+      <xacro:insert_block name="origin"/>
+      <axis xyz="0 0 1"/>
+      <limit effort="6" velocity="${vlimit}" lower="${llimit}" upper="${ulimit}"/>
+      <dynamics friction="0.13"/>
+      <parent link="${parent}"/>
+      <child link="${name}_link"/>
+    </joint>
+    <link name="${name}_link">
+      <!-- TODO: This inertial field needs doesn't contain reliable data!! -->
+      <inertial>
+        <mass value="0.008"/>
+        <origin xyz="0 0 0"/>
+        <inertia ixx="0.000001" ixy="0.0" ixz="0.0"
+                 iyy="0.000001" iyz="0.0"
+                 izz="0.000001"/>
+      </inertial>
+      <visual>
+        <origin xyz="0 0 0" rpy="0 0 0"/>
+        <geometry>
+          <mesh filename="package://phantomx_pincher_arm_description/meshes/F2Bracket.stl" scale="1.0 1.0 1.0"/>
+        </geometry>
+        <material name="${color}"/>
+      </visual>
+      <collision>
+        <origin xyz="0 0 0" rpy="0 0 0"/>
+        <geometry>
+          <mesh filename="package://phantomx_pincher_arm_description/meshes/F2Bracket.stl" scale="1.0 1.0 1.0"/>
+        </geometry>
+      </collision>
+    </link>
+    <gazebo reference="${name}_link">
+      <material>Gazebo/${color}</material>
+      <gravity>true</gravity>
+    </gazebo>
+  </xacro:macro>
+  <xacro:macro name="pincher_bicep" params="parent name color llimit ulimit vlimit *origin">
+    <joint name="${name}_joint" type="revolute">
+      <xacro:insert_block name="origin"/>
+      <axis xyz="0 1 0"/>
+      <limit effort="6" velocity="${vlimit}" lower="${llimit}" upper="${ulimit}"/>
+      <dynamics friction="0.13"/>
+      <parent link="${parent}"/>
+      <child link="${name}_link"/>
+    </joint>
+    <link name="${name}_link">
+      <!-- TODO: This inertial field needs doesn't contain reliable data!! -->
+      <inertial>
+        <mass value="0.016"/>
+        <origin xyz="0 0 0"/>
+        <inertia ixx="0.000001" ixy="0.0" ixz="0.0"
+                 iyy="0.000001" iyz="0.0"
+                 izz="0.000001"/>
+      </inertial>
+      <visual>
         <origin xyz=" 0 0 0 " rpy="0 0 0"/>
         <geometry>
-          <mesh filename="package://phantomx_pincher_arm_description/meshes/ax12_box.stl" scale="${M_SCALE} ${M_SCALE} ${M_SCALE}"/>
-        </geometry>
-        <material name="Black"/>
-      </visual>
-      <collision>
-        <origin xyz="0.0 0.0 -0.01241" rpy="0 0 0"/>
-        <geometry>
-          <box size="0.025 0.038 0.04762"/>
-        </geometry>
-      </collision>
-    </link>
-    <gazebo reference="${name}_link">
-      <material>Gazebo/Black</material>
-      <selfCollide>true</selfCollide>
-      <gravity>true</gravity>
-    </gazebo>
-  </xacro:macro>
-  <xacro:macro name="bioloid_F10_fixed" params="parent name color *origin">
-    <joint name="${name}_joint" type="fixed">
-      <insert_block name="origin"/>
-      <parent link="${parent}"/>
-      <child link="${name}_link"/>
-    </joint>
-    <link name="${name}_link">
-      <inertial>
-        <mass value="0.004"/>
+          <mesh filename="package://phantomx_pincher_arm_description/meshes/PincherBicep.stl" scale="1.0 1.0 1.0"/>
+        </geometry>
+        <material name="${color}"/>
+      </visual>
+      <collision>
+        <origin xyz="0.0 0.0 0.0" rpy="0 0 0"/>
+        <geometry>
+          <mesh filename="package://phantomx_pincher_arm_description/meshes/PincherBicep.stl" scale="1.0 1.0 1.0"/>
+        </geometry>
+      </collision>
+    </link>
+    <gazebo reference="${name}_link">
+      <material>Gazebo/${color}</material>
+      <gravity>true</gravity>
+    </gazebo>
+  </xacro:macro>
+  <xacro:macro name="pincher_forearm" params="parent name color llimit ulimit vlimit *origin">
+    <joint name="${name}_joint" type="revolute">
+      <xacro:insert_block name="origin"/>
+      <axis xyz="0 -1 0"/>
+      <limit effort="6" velocity="${vlimit}" lower="${llimit}" upper="${ulimit}"/>
+      <dynamics friction="0.13"/>
+      <parent link="${parent}"/>
+      <child link="${name}_link"/>
+    </joint>
+    <link name="${name}_link">
+      <!-- TODO: This inertial field needs doesn't contain reliable data!! -->
+      <inertial>
+        <mass value="0.016"/>
         <origin xyz="0 0 0"/>
         <inertia ixx="0.000001" ixy="0.0" ixz="0.0"
@@ -96,5 +132,5 @@
         <origin xyz=" 0 0 0 " rpy="0 0 0"/>
         <geometry>
-          <mesh filename="package://phantomx_pincher_arm_description/meshes/F10.stl" scale="${M_SCALE} ${M_SCALE} ${M_SCALE}"/>
+          <mesh filename="package://phantomx_pincher_arm_description/meshes/PincherForeArm.stl" scale="1.0 1.0 1.0"/>
         </geometry>
         <material name="${color}"/>
@@ -103,23 +139,26 @@
         <origin xyz="0.0 0.0 0.0" rpy="0 0 0"/>
         <geometry>
-          <box size="0.025 0.038 0.004"/>
-        </geometry>
-      </collision>
-    </link>
-    <gazebo reference="${name}_link">
-      <material>Gazebo/${color}</material>
-      <selfCollide>true</selfCollide>
-      <gravity>true</gravity>
-    </gazebo>
-  </xacro:macro>
-  <xacro:macro name="bioloid_F3_fixed" params="parent name color *origin">
-    <joint name="${name}_joint" type="fixed">
-      <insert_block name="origin"/>
-      <parent link="${parent}"/>
-      <child link="${name}_link"/>
-    </joint>
-    <link name="${name}_link">
-      <inertial>
-        <mass value="0.005"/>
+          <mesh filename="package://phantomx_pincher_arm_description/meshes/PincherForeArm.stl" scale="1.0 1.0 1.0"/>
+        </geometry>
+      </collision>
+    </link>
+    <gazebo reference="${name}_link">
+      <material>Gazebo/${color}</material>
+      <gravity>true</gravity>
+    </gazebo>
+  </xacro:macro>
+  <xacro:macro name="pincher_wrist" params="parent name color llimit ulimit vlimit *origin">
+    <joint name="${name}_joint" type="revolute">
+      <xacro:insert_block name="origin"/>
+      <axis xyz="0 -1 0"/>
+      <limit effort="6" velocity="${vlimit}" lower="${llimit}" upper="${ulimit}"/>
+      <dynamics friction="0.13"/>
+      <parent link="${parent}"/>
+      <child link="${name}_link"/>
+    </joint>
+    <link name="${name}_link">
+      <!-- TODO: This inertial field needs doesn't contain reliable data!! -->
+      <inertial>
+        <mass value="0.01"/>
         <origin xyz="0 0 0"/>
         <inertia ixx="0.000001" ixy="0.0" ixz="0.0"
@@ -130,192 +169,47 @@
         <origin xyz=" 0 0 0 " rpy="0 0 0"/>
         <geometry>
-          <mesh filename="package://phantomx_pincher_arm_description/meshes/F3.stl" scale="${M_SCALE} ${M_SCALE} ${M_SCALE}"/>
-        </geometry>
-        <material name="${color}"/>
-      </visual>
-      <collision>
-        <origin xyz="0.0 0.0 -0.0045" rpy="0 0 0"/>
-        <geometry>
-          <box size="0.025 0.038 0.009"/>
-        </geometry>
-      </collision>
-    </link>
-    <gazebo reference="${name}_link">
-      <material>Gazebo/${color}</material>
-      <selfCollide>true</selfCollide>
-      <gravity>true</gravity>
-    </gazebo>
-  </xacro:macro>
-  <xacro:macro name="bioloid_F3_revolute" params="parent name color llimit ulimit vlimit *origin">
-    <joint name="${name}_joint" type="revolute">
-      <insert_block name="origin"/>
-      <axis xyz="0 0 -1"/>
-      <limit effort="30" velocity="${vlimit}" lower="${llimit}" upper="${ulimit}"/>
-      <dynamics friction="0.13"/>
-      <parent link="${parent}"/>
-      <child link="${name}_link"/>
-    </joint>
-    <link name="${name}_link">
-      <inertial>
-        <mass value="0.008"/>
-        <origin xyz="0 0 0"/>
-        <inertia ixx="0.000001" ixy="0.0" ixz="0.0"
-                 iyy="0.000001" iyz="0.0"
-                 izz="0.000001"/>
-      </inertial>
-      <visual>
-        <origin xyz=" 0 0 0 " rpy="0 0 0"/>
-        <geometry>
-          <mesh filename="package://phantomx_pincher_arm_description/meshes/F3.stl" scale="${M_SCALE} ${M_SCALE} ${M_SCALE}"/>
-        </geometry>
-        <material name="${color}"/>
-      </visual>
-      <collision>
-        <origin xyz="0.0 0.0 -0.0045" rpy="0 0 0"/>
-        <geometry>
-          <box size="0.025 0.038 0.009"/>
-        </geometry>
-      </collision>
-    </link>
-    <gazebo reference="${name}_link">
-      <material>Gazebo/${color}</material>
-      <selfCollide>true</selfCollide>
-      <gravity>true</gravity>
-    </gazebo>
-  </xacro:macro>
-  <xacro:macro name="bioloid_F2_revolute" params="parent name color llimit ulimit vlimit *origin">
-    <joint name="${name}_joint" type="revolute">
-      <insert_block name="origin"/>
-      <axis xyz="0 1 0"/>
-      <limit effort="30" velocity="${vlimit}" lower="${llimit}" upper="${ulimit}"/>
-      <dynamics friction="0.13"/>
-      <parent link="${parent}"/>
-      <child link="${name}_link"/>
-    </joint>
-    <link name="${name}_link">
-      <inertial>
-        <mass value="0.010"/>
-        <origin xyz="0 0 0"/>
-        <inertia ixx="0.000001" ixy="0.0" ixz="0.0"
-                 iyy="0.000001" iyz="0.0"
-                 izz="0.000001"/>
-      </inertial>
-      <visual>
-        <origin xyz=" 0 0 0 " rpy="0 0 0"/>
-        <geometry>
-          <mesh filename="package://phantomx_pincher_arm_description/meshes/F2.stl" scale="${M_SCALE} ${M_SCALE} ${M_SCALE}"/>
-        </geometry>
-        <material name="${color}"/>
-      </visual>
-      <collision>
-        <origin xyz="0.0 0.0 0.00775" rpy="0 0 0"/>
-        <geometry>
-          <box size="0.025 0.0485 0.0375"/>
-        </geometry>
-      </collision>
-    </link>
-    <gazebo reference="${name}_link">
-      <material>Gazebo/${color}</material>
-      <selfCollide>true</selfCollide>
-      <gravity>true</gravity>
-    </gazebo>
-  </xacro:macro>
-  <xacro:macro name="bioloid_F4_revolute" params="parent name color llimit ulimit vlimit *origin">
-    <joint name="${name}_joint" type="revolute">
-      <insert_block name="origin"/>
-      <axis xyz="0 1 0"/>
-      <limit effort="30" velocity="${vlimit}" lower="${llimit}" upper="${ulimit}"/>
-      <dynamics friction="0.13"/>
-      <parent link="${parent}"/>
-      <child link="${name}_link"/>
-    </joint>
-    <link name="${name}_link">
-      <inertial>
-        <mass value="0.016"/>
-        <origin xyz="0 0 0"/>
-        <inertia ixx="0.000001" ixy="0.0" ixz="0.0"
-                 iyy="0.000001" iyz="0.0"
-                 izz="0.000001"/>
-      </inertial>
-      <visual>
-        <origin xyz=" 0 0 0 " rpy="0 0 0"/>
-        <geometry>
-          <mesh filename="package://phantomx_pincher_arm_description/meshes/F4.stl" scale="${M_SCALE} ${M_SCALE} ${M_SCALE}"/>
-        </geometry>
-        <material name="${color}"/>
-      </visual>
-      <collision>
-        <origin xyz="0.0 0.0 0.0215" rpy="0 0 0"/>
-        <geometry>
-          <box size="0.028 0.0485 0.065"/>
-        </geometry>
-      </collision>
-    </link>
-    <gazebo reference="${name}_link">
-      <material>Gazebo/${color}</material>
-      <selfCollide>true</selfCollide>
-      <gravity>true</gravity>
-    </gazebo>
-  </xacro:macro>
-  <xacro:macro name="gripper_finger_base" params="parent name color *origin">
-    <joint name="${name}_joint" type="fixed">
-      <insert_block name="origin"/>
-      <parent link="${parent}"/>
-      <child link="${name}_link"/>
-    </joint>
-    <link name="${name}_link">
-      <inertial>
-        <mass value="0.00001"/>
-        <origin xyz="0 0 0"/>
-        <inertia ixx="1.0" ixy="0.0" ixz="0.0"
-          iyy="1.0" iyz="0.0"
-          izz="1.0"/>
-      </inertial>
-      <visual>
-        <origin xyz="0.016 0 -.015 " rpy="${M_PI} ${-M_PI/2} ${M_PI/2}"/>
-        <geometry>
-          <mesh filename="package://phantomx_pincher_arm_description/meshes/pincher_finger_base.stl" scale=".01 .01 .01"/>
-        </geometry>
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
File: phantomx_pincher_arm_description/urdf/phantomx_pincher_arm.urdf.xacro (robot description, xacro)
@@ -3,21 +3,21 @@
 <robot name="phantomx_pincher_arm" xmlns:xacro="http://ros.org/wiki/xacro">
     <!-- We can configure joints velocity limit and lower/upper limits
-          to allow access to different operational areas, e.g. left handed vs. right handed robot -->
+    to allow access to different operational areas, e.g. left handed vs. right handed robot -->
     <xacro:property name="joints_vlimit" value="1.571"/>
-    <xacro:property name="pan_llimit" value="-2.617"/>
-    <xacro:property name="pan_ulimit" value="2.617"/>
-    <xacro:property name="shoulder_llimit" value="-2.2"/>
-    <xacro:property name="shoulder_ulimit" value="2.16"/>
-    <xacro:property name="elbow_llimit" value="-2.42"/>
-    <xacro:property name="elbow_ulimit" value="2.38"/>
-    <xacro:property name="wrist_llimit" value="-1.72"/>
-    <xacro:property name="wrist_ulimit" value="1.68"/>
+    <xacro:property name="pan_llimit" value="-1.74"/>
+    <xacro:property name="pan_ulimit" value="1.74"/>
+    <xacro:property name="shoulder_llimit" value="-1.98"/>
+    <xacro:property name="shoulder_ulimit" value="1.88"/>
+    <xacro:property name="elbow_llimit" value="-1.58"/>
+    <xacro:property name="elbow_ulimit" value="0.59"/>
+    <xacro:property name="wrist_llimit" value="-1.79"/>
+    <xacro:property name="wrist_ulimit" value="1.67"/>
     <!-- Included URDF Files -->
     <xacro:include filename="$(find phantomx_pincher_arm_description)/urdf/phantomx_pincher_arm.xacro"/>
     <!-- As we don't have a base here, add a base_link link as location reference -->
     <link name="base_link"/>
-    <!-- phantomx_pincher_arm macro -->
-    <phantomx_pincher_arm parent="base_link" color="Gray" gripper_color="Gray">
-      <origin xyz="0.1 0.03 0.435"/>
+    <!-- phantomx_pincher_arm macro //joints_vlimit="${joints_vlimit}" pan_llimit="-2.617" pan_ulimit="2.617// -->
+    <phantomx_pincher_arm parent="base_link" color="White" gripper_color="White">
+        <origin xyz="0.12 0.00 0.140"/>
     </phantomx_pincher_arm>
 </robot>
