Commit message: Pincher MK3 Updates. New IKFast solver.

File: phantomx_pincher_arm_description/urdf/phantomx_pincher_arm.xacro (robot description, xacro)
@@ -1,94 +1,93 @@
 <?xml version="1.0"?>
 <!-- Arm description for PhantomX Pincher arm -->
-<robot xmlns:xacro="http://ros.org/wiki/xacro">
+<robot name="phantomx_pincher_arm" xmlns:xacro="http://ros.org/wiki/xacro">
   <xacro:include filename="$(find phantomx_pincher_arm_description)/urdf/arm_hardware.xacro"/>
-  <material name="White">
-    <color rgba="0.87 0.90 0.87 1.0"/>
-  </material>
-  <material name="Black">
-    <color rgba="0.08 0.08 0.08 1.0"/>
-  </material>
-  <material name="Gray">
-    <color rgba="0.2 0.2 0.21 1.0"/>
-  </material>
-  <material name="Green">
-    <color rgba="0.22 0.32 0.14 1.0"/>
-  </material>
+  <!--joints_vlimit pan_llimit pan_ulimit-->
   <xacro:macro name="phantomx_pincher_arm" params="parent color gripper_color *origin">
-    <link name="arm_base_link"/>
-    <joint name="arm_base_joint" type="fixed">
-      <insert_block name="origin"/>
-      <parent link="${parent}"/>
-      <child link="arm_base_link"/>
-    </joint>
-    <!-- fake gripper_link joint gives us a free servo!
-         this makes us 5DOF and saves you $44.90
-         that's a lot of coin! -->
+    <!-- arm base link -->
+    <pincher_base parent="${parent}" name="arm_base">
+      <xacro:insert_block name="origin"/>
+    </pincher_base>
+    <bracket_F2_revolute parent="arm_base_link" name="arm_shoulder_pan" color="${color}"
+                         vlimit="${joints_vlimit}" llimit="${pan_llimit}" ulimit="${pan_ulimit}">
+      <origin xyz="0 0 0.020" rpy="0 0 0"/>
+    </bracket_F2_revolute>
+    <transmission name="arm_shoulder_pan_transmission">
+      <type>transmission_interface/SimpleTransmission</type>
+      <joint name="arm_shoulder_pan_joint">
+        <hardwareInterface>EffortJointInterface</hardwareInterface>
+      </joint>
+      <actuator name="arm_shoulder_pan_actuator">
+        <hardwareInterface>EffortJointInterface</hardwareInterface>
+        <mechanicalReduction>1</mechanicalReduction>
+      </actuator>
+    </transmission>
+    <!-- shoulder lift joint -->
+    <pincher_bicep parent="arm_shoulder_pan_link" name="arm_bicep" color="${color}"
+                         vlimit="${joints_vlimit}" llimit="${shoulder_llimit}" ulimit="${shoulder_ulimit}">
+      <origin xyz="0 0 0.027" rpy="0 0 0"/>
+    </pincher_bicep>
+    <transmission name="arm_bicep_transmission">
+      <type>transmission_interface/SimpleTransmission</type>
+      <joint name="arm_bicep_joint">
+        <hardwareInterface>EffortJointInterface</hardwareInterface>
+      </joint>
+      <actuator name="arm_bicep_actuator">
+        <hardwareInterface>EffortJointInterface</hardwareInterface>
+        <mechanicalReduction>1</mechanicalReduction>
+      </actuator>
+    </transmission>
+    <!-- elbow joint -->
+    <pincher_forearm parent="arm_bicep_link" name="arm_forearm" color="${color}"
+                         vlimit="${joints_vlimit}" llimit="${elbow_llimit}" ulimit="${elbow_ulimit}">
+      <origin xyz="0.0325 0 0.104" rpy="0 0 0"/>
+    </pincher_forearm>
+    <transmission name="arm_forearm_transmission">
+      <type>transmission_interface/SimpleTransmission</type>
+      <joint name="arm_forearm_joint">
+        <hardwareInterface>EffortJointInterface</hardwareInterface>
+      </joint>
+      <actuator name="arm_forearm_actuator">
+        <hardwareInterface>EffortJointInterface</hardwareInterface>
+        <mechanicalReduction>1</mechanicalReduction>
+      </actuator>
+    </transmission>
+    <!-- wrist joint -->
+    <pincher_wrist parent="arm_forearm_link" name="arm_wrist_flex" color="${color}"
+                         vlimit="${joints_vlimit}" llimit="${wrist_llimit}" ulimit="${wrist_ulimit}">
+      <origin xyz="0.104 0 0" rpy="0 0 0"/>
+    </pincher_wrist>
+    <transmission name="arm_wrist_flex_transmission">
+      <type>transmission_interface/SimpleTransmission</type>
+      <joint name="arm_wrist_flex_joint">
+        <hardwareInterface>EffortJointInterface</hardwareInterface>
+      </joint>
+      <actuator name="arm_wrist_flex_actuator">
+        <hardwareInterface>EffortJointInterface</hardwareInterface>
+        <mechanicalReduction>1</mechanicalReduction>
+      </actuator>
+    </transmission>
+  <!-- gripper -->
+  <xacro:include filename="$(find phantomx_pincher_arm_description)/urdf/phantomx_pincher_gripper.xacro"/>
+<!-- gripper_link -->
     <link name="gripper_link"/>
     <joint name="gripper_link_joint" type="revolute">
-      <origin xyz="0 0 0.112" rpy="0 -1.57 0"/>
+      <origin xyz="0.110 0 0" rpy="0 0 0"/>
       <parent link="arm_wrist_flex_link"/>
       <child link="gripper_link"/>
-      <limit effort="30" velocity="1" lower="-3.14" upper="3.14"/>
+      <limit effort="6" velocity="1" lower="-3.14" upper="3.14"/>
       <axis xyz="1 0 0"/>
     </joint>
-    <!-- shoulder pan joint -->
-    <dynamixel_AX12_fixed parent="arm_base_link" name="arm_shoulder_pan_servo">
-      <origin xyz="0 0 0" rpy="${M_PI/2} 0 ${M_PI/2}"/>
-    </dynamixel_AX12_fixed>
-    <bioloid_F3_revolute parent="arm_shoulder_pan_servo_link" name="arm_shoulder_pan" color="${color}"
-                         vlimit="${joints_vlimit}" llimit="${pan_llimit}" ulimit="${pan_ulimit}">
-      <origin xyz="0 ${AX12_WIDTH/2} 0" rpy="${-M_PI/2} ${M_PI/2} ${M_PI}"/>
-    </bioloid_F3_revolute>
-    <!-- shoulder lift joint -->
-    <dynamixel_AX12_fixed parent="arm_shoulder_pan_link" name="arm_shoulder_lift_servo">
-      <origin xyz="0 0 ${-AX12_HEIGHT-F10_HEIGHT+0.001}" rpy="0 ${M_PI} 0"/>
-    </dynamixel_AX12_fixed>
-    <bioloid_F4_revolute parent="arm_shoulder_lift_servo_link" name="arm_shoulder_lift" color="${color}"
-                         vlimit="${joints_vlimit}" llimit="${shoulder_llimit}" ulimit="${shoulder_ulimit}">
-      <origin xyz="0 0 0" rpy="0 0 0"/>
-    </bioloid_F4_revolute>
-    <bioloid_F10_fixed parent="arm_shoulder_lift_link" name="arm_shoulder_F10_0" color="${color}">
-      <origin xyz="0 0 ${F4_HEIGHT+F10_HEIGHT/2}" rpy="0 0 0"/>
-    </bioloid_F10_fixed>
-    <bioloid_F10_fixed parent="arm_shoulder_F10_0_link" name="arm_shoulder_F10_1" color="${color}">
-      <origin xyz="0 0 ${F10_HEIGHT}" rpy="0 0 0"/>
-    </bioloid_F10_fixed>
-    <bioloid_F10_fixed parent="arm_shoulder_F10_1_link" name="arm_shoulder_F10_2" color="${color}">
-      <origin xyz="0 0 ${F10_HEIGHT}" rpy="0 0 0"/>
-    </bioloid_F10_fixed>
-    <bioloid_F3_fixed parent="arm_shoulder_F10_2_link" name="arm_shoulder_F3_0" color="${color}">
-      <origin xyz="0 0 ${F10_HEIGHT/2}" rpy="0 ${M_PI} 0"/>
-    </bioloid_F3_fixed>
-    <!-- elbow joint -->
-    <dynamixel_AX12_fixed parent="arm_shoulder_F3_0_link" name="arm_elbow_flex_servo">
-      <origin xyz="0 0 ${-AX12_HEIGHT-F10_HEIGHT+0.001}" rpy="0 ${M_PI} 0"/>
-    </dynamixel_AX12_fixed>
-    <bioloid_F4_revolute parent="arm_elbow_flex_servo_link" name="arm_elbow_flex" color="${color}"
-                         vlimit="${joints_vlimit}" llimit="${elbow_llimit}" ulimit="${elbow_ulimit}">
-      <origin xyz="0 0 0" rpy="0 0 0"/>
-    </bioloid_F4_revolute>
-    <bioloid_F10_fixed parent="arm_elbow_flex_link" name="arm_elbow_F10_0" color="${color}">
-      <origin xyz="0 0 ${F4_HEIGHT+F10_HEIGHT/2}" rpy="0 0 0"/>
-    </bioloid_F10_fixed>
-    <bioloid_F10_fixed parent="arm_elbow_F10_0_link" name="arm_elbow_F10_1" color="${color}">
-      <origin xyz="0 0 ${F10_HEIGHT}" rpy="0 0 0"/>
-    </bioloid_F10_fixed>
-    <bioloid_F10_fixed parent="arm_elbow_F10_1_link" name="arm_elbow_F10_2" color="${color}">
-      <origin xyz="0 0 ${F10_HEIGHT}" rpy="0 0 0"/>
-    </bioloid_F10_fixed>
-    <bioloid_F3_fixed parent="arm_elbow_F10_2_link" name="arm_elbow_F3_0" color="${color}">
-      <origin xyz="0 0 ${F10_HEIGHT/2}" rpy="0 ${M_PI} 0"/>
-    </bioloid_F3_fixed>
-    <!-- wrist joint -->
-    <dynamixel_AX12_fixed parent="arm_elbow_F3_0_link" name="arm_wrist_flex_servo">
-      <origin xyz="0 0 ${-AX12_HEIGHT-F10_HEIGHT+0.001}" rpy="0 ${M_PI} 0"/>
-    </dynamixel_AX12_fixed>
-    <bioloid_F2_revolute parent="arm_wrist_flex_servo_link" name="arm_wrist_flex" color="${color}"
-                         vlimit="${joints_vlimit}" llimit="${wrist_llimit}" ulimit="${wrist_ulimit}">
-      <origin xyz="0 0 0" rpy="0 0 0"/>
-    </bioloid_F2_revolute>
-  <!-- gripper -->
-  <xacro:include filename="$(find phantomx_pincher_arm_description)/urdf/phantomx_pincher_gripper.xacro"/>
+  <!--gazebo>
+      <gripper name="gripper">
+        <grasp_check>
+          <attach_steps>5</attach_steps>
+          <detach_steps>10</detach_steps>
+          <min_contact_count>2</min_contact_count>
+        </grasp_check>
+      </gripper>
+      <gripper_link>gripper_active_link</gripper_link>
+      <palm_link>gripper_servo_link</palm_link>
+  </gazebo-->
   </xacro:macro>
 </robot>

File: phantomx_pincher_arm_description/urdf/phantomx_pincher_gripper.xacro (robot description, xacro)
@@ -1,45 +1,37 @@
 <?xml version="1.0"?>
-<!-- PhantomX Pincher Arm gripper URDF-->
+<!-- PhantomX Pincher gripper URDF-->
 <robot xmlns:xacro="http://ros.org/wiki/xacro">
-    <bioloid_F3_fixed parent="arm_wrist_flex_link" name="arm_wrist_F3_0" color="${color}">
-      <origin xyz="0 0 ${F2_HEIGHT}" rpy="0 ${M_PI} ${-M_PI}"/>
-    </bioloid_F3_fixed>
     <!-- gripper joint -->
-    <dynamixel_AX12_fixed parent="arm_wrist_F3_0_link" name="gripper_servo" >
-      <origin xyz="0 0 ${-AX12_WIDTH/2}" rpy="${M_PI/2} ${M_PI} ${M_PI/2}"/>
-    </dynamixel_AX12_fixed>
-     <gripper_finger_base parent="gripper_servo_link" name="gripper_finger_base" color="${color}">
-      <origin xyz="0.01  ${AX12_WIDTH} 0" rpy="${M_PI/2} ${-M_PI} ${M_PI/2}"/>
-    </gripper_finger_base>
-     <!-- Finger 1 -->
+    <!-- Finger 1 -->
     <joint name="gripper_joint" type="prismatic">
-      <origin xyz="0 0 0" rpy="0 0 0"/>
-      <axis xyz="1 0 0"/>
-      <limit effort="30" velocity="0.5" lower="0.002" upper="0.031"/>
-      <parent link="gripper_servo_link"/>
+      <origin xyz="0.070 0 0" rpy="0 0 0"/>
+      <axis xyz="0 1 0"/>
+      <limit effort="30" velocity="0.5" lower="0.002" upper="0.032"/>
+      <parent link="arm_wrist_flex_link"/>
       <child link="gripper_active_link"/>
     </joint>
-    <phantomx_pincher_gripper name="gripper_active" color="${color}" >
-      <origin xyz="-0.02 0.023 0" rpy="${-M_PI/2} 0 0"/>
-    </phantomx_pincher_gripper>
+    <pincher_finger name="gripper_active" color="${color}" >
+      <origin xyz="0 0 0" rpy="0 0 0"/>
+    </pincher_finger>
     <!-- Finger 2 -->
     <!-- Note: currently static but should be a Mimic of Finger 1 -->
     <joint name="gripper2_joint" type="fixed">
-      <parent link="gripper_servo_link"/>
+      <origin xyz="0.070 -0.016 0" rpy="0 0 0"/>
+      <parent link="arm_wrist_flex_link"/>
       <child link="gripper_active2_link"/>
     </joint>
-    <phantomx_pincher_gripper name="gripper_active2" color="${color}" >
-      <origin xyz="-0.02 0.023 0" rpy="${-M_PI/2} ${M_PI} 0"/>
-    </phantomx_pincher_gripper>
+    <pincher_finger name="gripper_active2" color="${color}" >
+      <origin xyz="0 0 0" rpy="${M_PI} 0 0"/>
+    </pincher_finger>
     <!-- Using Mimic -->
     <!-- gripper 2 joint -->
-    <!--  ### Mimic would be better but causes Missing Joint error in Moveit
-      <joint name="gripper2_joint" type="prismatic">
-      <origin xyz="0 0 0" rpy="0 0 0"/>
-      <axis xyz="0 0 1"/>
-      <limit effort="30" velocity="0.5" lower="0.002" upper="0.031"/>
-      <parent link="gripper_servo_link"/>
+    <!--  TODO: Test Mimic ->
+    <joint name="gripper2_joint" type="prismatic">
+      <origin xyz="0.070 0 0" rpy="0 0 0"/>
+      <axis xyz="0 1 0"/>
+      <limit effort="30" velocity="0.5" lower="-0.016" upper="-0.002"/>
+      <parent link="arm_wrist_flex_link"/>
       <child link="gripper_active2_link"/>
-      <mimic joint="gripper_joint" multiplier="-.5"  offset = "0"/>
+      <mimic joint="gripper_joint" multiplier="-1"  offset = "0"/>
     </joint-->
 </robot>
