Commit message: Adjusting defaults

File: phantomx_pincher_arm_description/urdf/phantomx_pincher_arm.urdf.xacro (robot description, xacro)
@@ -19,5 +19,5 @@
     <!-- phantomx_pincher_arm macro //joints_vlimit="${joints_vlimit}" pan_llimit="-2.617" pan_ulimit="2.617// -->
     <phantomx_pincher_arm parent="base_link" color="White" gripper_color="White">
-        <origin xyz="0.12 0.00 0.140"/>
+        <origin xyz="0.0 0.00 0.077"/>
     </phantomx_pincher_arm>
 </robot>
